File: KiCad/RiscV_MousePcb.kicad_pcb (KiCad board)
At the start: 4 copper layers, 40.6 x 65.1 mm, 52 parts, among them J1 Conn_01x04_Pin, U1 TLV70019_SOT23-5, U2 MIC5219-3.3YM5, U3 CH32V30xRxTx, U4 TPD2EUSB30, U5 TPD2EUSB30, U6 TPD2EUSB30, Y1 8MHZ_CMOS

Commit message: Add files via upload
Parts:
- added REF**: MountingHole_3.2mm_M3, MountingHole:MountingHole_3.2mm_M3, F.Cu at (54.1, 77.6)
- added REF**: MountingHole_3.2mm_M3, MountingHole:MountingHole_3.2mm_M3, F.Cu at (54.5, 32.8)
- added REF**: MountingHole_3.2mm_M3, MountingHole:MountingHole_3.2mm_M3, F.Cu at (20.7, 77.3)
- added REF**: MountingHole_3.2mm_M3, MountingHole:MountingHole_3.2mm_M3, F.Cu at (21.0, 32.8)
- moved REF** 3.24 mm to (54.1, 77.6)
